File: my-keeb.kicad_pcb (KiCad board)
At the start: 2 copper layers, 190.5 x 95.2 mm, 108 parts, among them SW1 SW_Push, U1 ATmega32U4-AU, Y1 16MHz

Commit message: Routing in progress
Routing:
- net ROW3: track 0.00 -> 176.5 mm
- net ROW2: track 0.00 -> 176.5 mm
- net ROW1: track 0.00 -> 176.5 mm
- net ROW0: track 0.00 -> 176.5 mm
- net ROW4: track 0.00 -> 117.1 mm
- net COL7: track 0.00 -> 79.2 mm
- net COL6: track 0.00 -> 79.2 mm
- net COL3: track 0.00 -> 78.1 mm
- net COL2: track 0.00 -> 78.1 mm
- net COL5: track 0.00 -> 77.3 mm
- net COL4: track 0.00 -> 76.2 mm
- net COL1: track 0.00 -> 57.1 mm
- net COL9: track 0.00 -> 57.1 mm
- net COL8: track 0.00 -> 57.1 mm
- net COL0: track 0.00 -> 57.1 mm
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Other:
- net class Default: trace_width 0.25 -> 0.254
- net class Power added: clearance 0.2, trace_width 0.381, via_dia 0.8, via_drill 0.4

Commit message: Still working on routing
Parts:
- moved USB1 199.4 mm to (14.3, 97.6), turned to 0 degrees
- moved R1 29.9 mm to (175.4, 106.4), turned to 180 degrees
- moved F1 27.0 mm to (175.1, 90.3), turned to 180 degrees
- moved R2 26.4 mm to (175.4, 103.2), turned to 180 degrees
- moved R3 25.7 mm to (196.9, 87.7), turned to 0 degrees
- moved C3 24.2 mm to (199.6, 102.0), turned to 0 degrees
- moved C4 23.4 mm to (199.6, 93.7), turned to 180 degrees
- moved Y1 22.3 mm to (199.6, 97.9), turned to 90 degrees
- moved C5 21.4 mm to (196.9, 91.0), turned to 0 degrees
- moved R4 20.9 mm to (183.4, 106.7), turned to 0 degrees
- moved C1 19.7 mm to (192.4, 106.7), turned to 0 degrees
- moved C2 19.7 mm to (179.5, 101.3), turned to 90 degrees
- moved C7 19.2 mm to (180.0, 92.9), turned to 270 degrees
- moved C6 18.0 mm to (188.6, 87.8), turned to 180 degrees
- moved SW1 4.15 mm to (27.8, 93.7)
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Routing:
- net GND: track 24.2 -> 75.0 mm
- net +5V: track 0.00 -> 15.7 mm
- net Net-(C3-Pad1): track 3.13 -> 8.72 mm
- net Net-(C6-Pad1): track 0.00 -> 4.35 mm
- net Net-(R4-Pad2): track 0.00 -> 3.71 mm

Commit message: Still doing routing
Parts:
- moved R3 3.89 mm to (193.3, 89.2)
- moved C6 1.52 mm to (187.9, 89.2)
- moved C1 1.29 mm to (191.9, 105.5)
- moved R4 1.17 mm to (183.4, 105.5)
- moved C5 1.02 mm to (197.7, 91.6)
- moved C7 0.86 mm to (180.1, 93.7)
- moved C2 0.81 mm to (180.1, 100.8)
- moved C3 0.64 mm to (199.6, 102.7)
- moved Y1 0.44 mm to (199.6, 98.3)
- moved C4 0.32 mm to (199.6, 94.0)
Routing:
- net +5V: track 15.7 -> 48.2 mm, vias 0 -> 3
- net GND: track 75.0 -> 57.8 mm
- net Net-(C4-Pad1): track 11.4 -> 3.26 mm
- net Net-(R3-Pad2): track 0.00 -> 6.33 mm
- net Net-(C6-Pad1): track 4.35 -> 2.71 mm
- net Net-(R4-Pad2): track 3.71 -> 2.53 mm

Commit message: Working on matrix
Parts:
- moved USB1 199.2 mm to (201.6, 29.9), turned to 180 degrees
- moved SW1 170.3 mm to (197.9, 86.0), turned to 0 degrees
- moved R1 19.6 mm to (183.9, 88.6), turned to 90 degrees
- moved R2 18.1 mm to (186.2, 88.6), turned to 90 degrees
- moved F1 6.35 mm to (181.5, 90.3), turned to 90 degrees
- moved C1 5.74 mm to (197.6, 106.0), turned to 90 degrees
- moved R4 5.66 mm to (178.2, 103.3), turned to 270 degrees
- moved C2 2.10 mm to (181.0, 102.7), turned to 180 degrees
- moved C3 1.69 mm to (201.0, 103.6)
- moved U1 1.66 mm to (189.6, 98.2)
- moved C5 1.66 mm to (199.1, 92.5)
- moved R3 1.66 mm to (194.7, 90.0)
- moved C7 1.66 mm to (181.5, 94.6)
- moved Y1 1.66 mm to (201.0, 99.2)
- moved C4 1.59 mm to (201.0, 94.7)
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Connections:
- U1 pad 22: Net-(U1-Pad22) -> ROW4
- U1 pad 25: Net-(U1-Pad25) -> COL0
- U1 pad 26: Net-(U1-Pad26) -> COL1
- U1 pad 27: Net-(U1-Pad27) -> COL2
- U1 pad 28: Net-(U1-Pad28) -> COL3
- U1 pad 29: Net-(U1-Pad29) -> COL4
- U1 pad 30: Net-(U1-Pad30) -> COL5
- U1 pad 31: Net-(U1-Pad31) -> COL6
- U1 pad 32: Net-(U1-Pad32) -> COL7
- U1 pad 36: Net-(U1-Pad36) -> ROW3
- U1 pad 37: Net-(U1-Pad37) -> ROW2
- U1 pad 38: Net-(U1-Pad38) -> ROW1
- U1 pad 39: Net-(U1-Pad39) -> ROW0
- U1 pad 40: Net-(U1-Pad40) -> COL8
- U1 pad 41: Net-(U1-Pad41) -> COL9
Routing:
- net GND: track 57.8 -> 145.8 mm, vias 0 -> 2
- net ROW0: track 176.5 -> 263.1 mm, vias 0 -> 2
- net VCC: track 0.00 -> 72.9 mm, vias 0 -> 2
- net D-: track 0.00 -> 69.3 mm, vias 0 -> 2
- net D+: track 0.00 -> 67.4 mm, vias 0 -> 2
- net ROW1: track 176.5 -> 243.2 mm, vias 0 -> 2
- net ROW2: track 176.5 -> 223.3 mm, vias 0 -> 2
- net ROW3: track 176.5 -> 203.2 mm
- net Net-(USB1-Pad6): track 0.00 -> 16.3 mm
- net +5V: track 48.2 -> 59.2 mm
- net Net-(C4-Pad1): track 3.26 -> 11.6 mm, vias 0 -> 2
- net ROW4: track 117.1 -> 122.4 mm
- net Net-(R1-Pad1): track 0.00 -> 5.15 mm
- net Net-(R4-Pad2): track 2.53 -> 7.57 mm
- net Net-(R2-Pad1): track 0.00 -> 3.71 mm
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
Commit message: Finished routing
Parts:
- moved C1 2.29 mm to (199.9, 106.2), turned to 0 degrees
- moved C6 0.28 mm to (189.1, 89.4)
Connections:
- U1 pad 22: ROW4 -> Net-(U1-Pad22)
- U1 pad 36: ROW3 -> ROW4
- U1 pad 37: ROW2 -> ROW3
- U1 pad 38: ROW1 -> ROW2
- U1 pad 39: ROW0 -> ROW1
- U1 pad 40: COL8 -> ROW0
- U1 pad 41: COL9 -> COL8
- U1 pad 9: Net-(U1-Pad9) -> COL9
Routing:
- net COL0: track 57.1 -> 250.5 mm, vias 0 -> 1
- net COL1: track 57.1 -> 240.6 mm, vias 0 -> 1
- net COL2: track 78.1 -> 229.5 mm
- net COL3: track 78.1 -> 212.8 mm, vias 0 -> 1
- net COL4: track 76.2 -> 185.8 mm, vias 0 -> 1
- net COL5: track 77.3 -> 157.1 mm, vias 0 -> 1
- net COL6: track 79.2 -> 134.2 mm, vias 0 -> 1
- net COL7: track 79.2 -> 113.9 mm, vias 0 -> 1
- net COL8: track 57.1 -> 85.8 mm, vias 0 -> 1
- net COL9: track 57.1 -> 73.7 mm, vias 0 -> 1
- net ROW4: track 122.4 -> 128.2 mm
- net ROW0: track 263.1 -> 259.5 mm
- net GND: track 145.8 -> 142.2 mm
- net ROW3: track 203.2 -> 205.6 mm
- net ROW1: track 243.2 -> 241.5 mm
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
Commit message: Finished designing the pcb!
Parts:
- moved C3 1.99 mm to (199.3, 102.7)
- moved C4 1.66 mm to (199.4, 94.9)
- moved Y1 1.52 mm to (199.5, 99.2)
- moved C1 1.35 mm to (198.9, 105.3)
- moved F1 1.02 mm to (181.5, 89.3)
- moved C5 0.36 mm to (198.9, 92.2)
- moved R4 0.13 mm to (178.2, 103.1)
Routing:
- net +5V: track 59.8 -> 110.1 mm, vias 3 -> 0
- net Net-(C4-Pad1): track 11.6 -> 8.56 mm, vias 2 -> 0
- net GND: track 142.2 -> 144.9 mm
- net Net-(C3-Pad1): track 9.10 -> 6.79 mm
- added copper zone on B.Cu, net GND
Other:
- board text added: "Salsa"
