File: my-keeb-modular/my-keeb-2/my-keeb-2.kicad_pcb (KiCad board)
At the start: 2 copper layers, 95.2 x 95.2 mm, 46 parts

Commit message: Fixed track issues
Parts:
- added M1: 1x5, modular:1x5, F.Cu at (97.9, 38.2)
- added M2: 1x5, modular:1x5, F.Cu at (100.7, 38.2)
- added M3: 1x5, modular:1x5, F.Cu at (108.8, 41.8)
- added SW1: SW_Push, random-keyboard-parts:SKQG-1155865, F.Cu at (39.8, 44.4)
- added U1: ProMicro, Keebio-Parts:ArduinoProMicro-ZigZag, F.Cu at (54.9, 31.6)
Routing:
- net ROW4: track 64.7 -> 107.6 mm

Commit message: part2 wip routing
Parts:
- moved SW1 147.3 mm to (186.6, 31.8), turned to 270 degrees
- moved U1 119.7 mm to (174.6, 31.0), turned to 270 degrees
- moved M2 41.5 mm to (108.8, 78.9)
- moved M1 24.2 mm to (108.8, 59.8)
- moved D39 11.2 mm to (174.6, 30.2), turned to 180 degrees
- moved D40 11.2 mm to (174.6, 49.2), turned to 180 degrees
Routing:
- net COL6: track 88.8 -> 158.8 mm
- net COL5: track 91.1 -> 147.2 mm
- net COL7: track 108.4 -> 146.2 mm
- net COL9: track 130.2 -> 167.9 mm
- net GND: track 0.00 -> 34.9 mm
- net ROW0: track 57.2 -> 79.5 mm
- net ROW1: track 89.5 -> 110.9 mm
- net COL8: track 106.8 -> 124.4 mm
- net Net-(SW1-Pad1): track 0.00 -> 14.6 mm
- net ROW3: track 43.5 -> 54.6 mm
- net ROW2: track 21.8 -> 32.7 mm
- net Net-(D40-Pad2): track 5.69 -> 13.0 mm
- net Net-(D39-Pad2): track 5.69 -> 13.0 mm
- net ROW4: track 107.6 -> 111.2 mm

Commit message: Finished modular pcb
Parts:
- removed SW1: SW_Push, random-keyboard-parts:SKQG-1155865
- moved D38 15.9 mm to (157.2, 98.4)
- moved D42 0.19 mm to (182.6, 79.4)
Routing:
- net COL0: track 0.00 -> 179.0 mm
- net COL1: track 0.00 -> 175.7 mm
- net COL2: track 0.00 -> 172.1 mm
- net COL3: track 0.00 -> 169.2 mm
- net COL4: track 0.00 -> 163.7 mm
- net ROW3: track 54.6 -> 149.3 mm
- net ROW2: track 32.7 -> 117.2 mm
- net ROW0: track 79.5 -> 140.9 mm
- net ROW4: track 111.2 -> 149.9 mm
- net Net-(SW1-Pad1): track 14.6 -> 0.00 mm
- net GND: track 34.9 -> 23.1 mm
- net COL5: track 147.2 -> 158.7 mm
- net COL6: track 158.8 -> 150.4 mm
- net Net-(D38-Pad2): track 5.69 -> 11.5 mm
- net Net-(D24-Pad2): track 0.00 -> 5.69 mm
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