File: my-keeb/my-keeb.sch (KiCad schematic (older format))
At the start: 108 parts, among them SW1 SW_Push, U1 ATmega32U4-AU, Y1 16MHz

Commit message: Improved USB routing for original my-keeb
Connections:
- net DN: now reaches R1.1, U1.3 (D-)
- net DP: now reaches R2.1, U1.4 (D+)
- no-connect marks 0 -> 1
Changed lines of the file:
@@
 Text GLabel 3350 6600 2    50   Input ~ 0
 COL8
+Text GLabel 1500 5300 3    50   Input ~ 0
+DN
+Text GLabel 1500 5200 1    50   Input ~ 0
+DP
+NoConn ~ 4250 7000
 $EndSCHEMATC
